File: PCB_PCB_Arduino_hot_gun_orig_2022-09-08.kicad_pcb (KiCad board)
At the start: 2 copper layers, 48.3 x 60.5 mm, 36 parts, among them M1 .Designator, Q1 IRFZ44NPBF, U1 TME 0505S, U2 ATMEGA328P-PU, U3 LM358, U4 1117-3.3, X1 16MHz

Commit message: note
Other:
- board text added: "Note: JST wire is usually mirrored, so the interface JST female header (right of the beeper) might need to be flipped. If soldered the plastic header part can be lifted and rotated without desoldering. Plugging in upside down won't cause any problem because the 24v relay is not enabled."
Changed lines of the file:
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@@
     (fp_arc (start 1.265 0.113) (mid -1.268817 -0.058661) (end 1.270126 0.000208) (layer "F.SilkS") (width 0.152))
     (fp_arc (start 4.814 -2.278) (mid 3.304871 -2.482691) (end 4.82623 -2.413163) (layer "F.SilkS") (width 0.152))
-    (fp_arc (start 5.998 0.132) (mid -5.999121 -0.072094) (end 5.999518 0.00018) (layer "F.SilkS") (width 0.152))
+    (fp_arc (start 5.998 0.132) (mid -5.999121 -0.072074) (end 5.999518 0.00018) (layer "F.SilkS") (width 0.152))
     (pad "" thru_hole circle locked (at -4.1 0 270) (size 2 2) (drill 1) (layers *.Cu *.Paste *.Mask)
       (net 10 "GND"))
@@
     (effects (font (size 2.032 2.032) (thickness 0.203)) (justify left))
   )
+  (gr_text "Note: JST wire is usually mirrored, so the interface JST female header (right of the beeper) might need to be flipped.\nIf soldered the plastic header part can be lifted and rotated without desoldering.\nPlugging in upside down won't cause any problem because the 24v relay is not enabled." (at 180.77 36.56) (layer "Cmts.User")
+    (effects (font (size 1.5 1.5) (thickness 0.25)))
+  )
   (dimension (type aligned) (layer "Dwgs.User")
